Commit message: setting base_footprint as robot root link

File: urdf/lucrezio_with_logical.urdf.xacro (robot description, xacro)
@@ -213,5 +213,5 @@
   <joint name="camera_joint" type="fixed">
     <axis xyz="0 1 0" />
-    <origin xyz="0 0 0.5" rpy="0 0 -1.57"/>
+    <origin xyz="0 0 0.5" rpy="0 0 0"/>
     <parent link="base_link"/>
     <child link="camera_link"/>
@@ -225,11 +225,11 @@
         <horizontal_fov>${60.0*M_PI/180.0}</horizontal_fov>
         <image>
-          <width>320</width>
-          <height>240</height>
+          <width>640</width>
+          <height>480</height>
           <format>R8G8B8</format>
         </image>
         <clip>
           <near>0.02</near>
-          <far>5.0</far>
+          <far>8.0</far>
         </clip>
       </camera>
@@ -278,5 +278,5 @@
   <joint name="logical_camera_joint" type="fixed">
     <axis xyz="0 1 0" />
-    <origin xyz="0 0 1.0" rpy="0 0 -1.57"/>
+    <origin xyz="0 0 1.0" rpy="0 0 0"/>
     <parent link="base_link"/>
     <child link="logical_camera_link"/>
@@ -288,5 +288,5 @@
           <logical_camera>
             <near>0.02</near>
-            <far>5.0</far>
+            <far>8.0</far>
             <horizontal_fov>${60.0*M_PI/180.0}</horizontal_fov>
             <aspect_ratio>1.778</aspect_ratio>
