Commit message: fixing annoying bugs ;)

File: urdf/lucrezio.urdf.xacro (robot description, xacro)
@@ -161,5 +161,5 @@
     <sensor type="gpu_ray" name="head_hokuyo_sensor">
       <pose>0 0 0 0 0 0</pose>
-      <visualize>true</visualize>
+      <visualize>false</visualize>
       <update_rate>40</update_rate>
       <ray>

File: urdf/lucrezio_with_logical.urdf.xacro (robot description, xacro)
@@ -161,5 +161,5 @@
     <sensor type="gpu_ray" name="head_hokuyo_sensor">
       <pose>0 0 0 0 0 0</pose>
-      <visualize>true</visualize>
+      <visualize>false</visualize>
       <update_rate>40</update_rate>
       <ray>
@@ -278,5 +278,5 @@
   <joint name="logical_camera_joint" type="fixed">
     <axis xyz="0 1 0" />
-    <origin xyz="0 0 1.0" rpy="0 0 0"/>
+    <origin xyz="0 0 0.5" rpy="0 0 0"/>
     <parent link="base_link"/>
     <child link="logical_camera_link"/>
@@ -292,5 +292,5 @@
             <aspect_ratio>1.778</aspect_ratio>
           </logical_camera>
-          <visualize>true</visualize>
+          <visualize>false</visualize>
           <always_on>true</always_on>
           <update_rate>10</update_rate>

Commit message: debugging

File: urdf/lucrezio.urdf.xacro (robot description, xacro)
@@ -166,12 +166,12 @@
         <scan>
           <horizontal>
-            <samples>720</samples>
+            <samples>1024</samples>
             <resolution>1</resolution>
-            <min_angle>-1.570796</min_angle>
-            <max_angle>1.570796</max_angle>
+            <min_angle>-1.57</min_angle>
+            <max_angle>1.57</max_angle>
           </horizontal>
         </scan>
         <range>
-          <min>0.10</min>
+          <min>0.02</min>
           <max>10.0</max>
           <resolution>0.01</resolution>
@@ -217,4 +217,7 @@
     <child link="camera_link"/>
   </joint>
+  <gazebo reference="camera_joint">
+    <preserveFixedJoint>true</preserveFixedJoint>
+  </gazebo>"
   <!-- XTION SENSOR -->
   <gazebo reference="camera_link">

File: urdf/lucrezio_with_logical.urdf.xacro (robot description, xacro)
@@ -210,4 +210,9 @@
     </inertial>
   </link>
+  <gazebo reference="camera_link">
+    <mu1>0.0</mu1>
+    <mu2>0.0</mu2>
+    <material>Gazebo/Black</material>
+  </gazebo>
   <!-- CAMERA JOINT -->
   <joint name="camera_joint" type="fixed">

Commit message: fixing stuff

File: urdf/lucrezio.urdf.xacro (robot description, xacro)
@@ -211,5 +211,5 @@
   </link>
   <!-- CAMERA JOINT -->
-  <joint name="camera_joint" type="fixed">
+  <joint name="camera_joint" type="continuous">
     <axis xyz="0 1 0" />
     <origin xyz="0 0 1.0" rpy="0 0 0"/>
@@ -217,7 +217,9 @@
     <child link="camera_link"/>
   </joint>
+<!--
   <gazebo reference="camera_joint">
     <preserveFixedJoint>true</preserveFixedJoint>
   </gazebo>"
+-->
   <!-- XTION SENSOR -->
   <gazebo reference="camera_link">

File: urdf/lucrezio_with_logical.urdf.xacro (robot description, xacro)
@@ -210,11 +210,6 @@
     </inertial>
   </link>
-  <gazebo reference="camera_link">
-    <mu1>0.0</mu1>
-    <mu2>0.0</mu2>
-    <material>Gazebo/Black</material>
-  </gazebo>
   <!-- CAMERA JOINT -->
-  <joint name="camera_joint" type="fixed">
+  <joint name="camera_joint" type="continuous">
     <axis xyz="0 1 0" />
     <origin xyz="0 0 0.5" rpy="0 0 0"/>
@@ -281,5 +276,5 @@
   </link>
   <!-- LOGICAL CAMERA JOINT -->
-  <joint name="logical_camera_joint" type="fixed">
+  <joint name="logical_camera_joint" type="continuous">
     <axis xyz="0 1 0" />
     <origin xyz="0 0 0.5" rpy="0 0 0"/>
